File: iGlass v1.brd (EAGLE design)
At the start: 86.4 x 22.9 mm, 13 parts, among them J1 1040310811, U1 ABX00027

Commit message: minor change to board
Routing:
- net PDM_DATA_2: track 75.5 -> 73.4 mm
- net GND: track 73.3 -> 73.4 mm, vias 13 -> 12
Changed lines of the file:
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@@
 <drawing>
 <settings>
-<setting alwaysvectorfont="yes"/>
+<setting alwaysvectorfont="no"/>
 <setting keepoldvectorfont="yes"/>
 <setting verticaltext="up"/>
@@
 <wire x1="81.56" y1="5.104" x2="82.574" y2="5.104" width="0.254" layer="1"/>
 <wire x1="82.574" y1="5.104" x2="84.074" y2="6.604" width="0.254" layer="1"/>
-<wire x1="50.924" y1="12.954" x2="51.054" y2="13.084" width="0.254" layer="1"/>
-<wire x1="51.054" y1="13.084" x2="51.054" y2="14.224" width="0.254" layer="1"/>
-<wire x1="51.054" y1="14.224" x2="51.562" y2="14.732" width="0.254" layer="1"/>
-<wire x1="51.562" y1="14.732" x2="52.832" y2="14.732" width="0.254" layer="1"/>
-<via x="52.832" y="14.732" extent="1-16" drill="0.6096"/>
 <wire x1="85.46" y1="9.404" x2="85.46" y2="7.99" width="0.254" layer="1"/>
 <wire x1="85.46" y1="7.99" x2="84.074" y2="6.604" width="0.254" layer="1"/>
@@
 <wire x1="52.9938" y1="10.414" x2="54.102" y2="10.414" width="1.016" layer="1"/>
 <via x="54.102" y="10.414" extent="1-16" drill="0.6096"/>
+<wire x1="50.924" y1="12.954" x2="52.9938" y2="10.8842" width="0.4064" layer="1"/>
+<wire x1="52.9938" y1="10.8842" x2="52.9938" y2="10.414" width="0.4064" layer="1"/>
 </signal>
 <signal name="VCC">
@@
 <wire x1="52.959" y1="17.24025" x2="52.959" y2="18.034" width="0.254" layer="1"/>
 <wire x1="52.959" y1="17.24025" x2="53.2765" y2="16.92275" width="0.254" layer="1"/>
-<wire x1="61.69025" y1="18.19275" x2="61.69025" y2="18.669" width="0.254" layer="1"/>
 <wire x1="52.959" y1="18.034" x2="52.824" y2="18.06" width="0.254" layer="1"/>
 <wire x1="61.69025" y1="18.19275" x2="61.714" y2="18.06" width="0.254" layer="1"/>
@@
 <wire x1="56.29275" y1="16.92275" x2="58.674" y2="19.304" width="0.254" layer="1"/>
 <wire x1="58.674" y1="19.304" x2="60.96" y2="19.304" width="0.254" layer="1"/>
+<wire x1="53.2765" y1="16.92275" x2="56.29275" y2="16.92275" width="0.254" layer="1"/>
+<wire x1="60.8965" y1="21.5265" x2="58.674" y2="19.304" width="0.254" layer="1"/>
 <wire x1="60.96" y1="19.304" x2="61.714" y2="18.55" width="0.254" layer="1"/>
 <wire x1="61.714" y1="18.55" x2="61.714" y2="18.06" width="0.254" layer="1"/>
-<wire x1="53.2765" y1="16.92275" x2="56.29275" y2="16.92275" width="0.254" layer="1"/>
-<wire x1="60.8965" y1="21.5265" x2="58.674" y2="19.304" width="0.254" layer="1"/>
 </signal>
 <signal name="SD_CD">
@@
 <wire x1="24.0665" y1="19.46275" x2="24.0665" y2="22.00275" width="0.254" layer="1"/>
 <wire x1="24.0665" y1="16.60525" x2="24.0665" y2="19.46275" width="0.254" layer="16"/>
-<wire x1="47.244" y1="16.60525" x2="24.0665" y2="16.60525" width="0.254" layer="1"/>
-<wire x1="47.244" y1="16.60525" x2="49.784" y2="14.06525" width="0.254" layer="1"/>
 <wire x1="24.0665" y1="22.00275" x2="23.974" y2="22.054" width="0.254" layer="1"/>
 <via x="65.50025" y="13.9065" extent="1-16" drill="0.6096"/>
@@
 <wire x1="66.802" y1="9.144" x2="66.04" y2="8.382" width="0.254" layer="16"/>
 <wire x1="66.04" y1="8.382" x2="66.04" y2="5.588" width="0.254" layer="16"/>
-<wire x1="65.50025" y1="13.9065" x2="65.50025" y2="12.92225" width="0.254" layer="1"/>
-<wire x1="63.754" y1="11.176" x2="65.50025" y2="12.92225" width="0.254" layer="1"/>
-<wire x1="65.50025" y1="10.69975" x2="65.50025" y2="12.92225" width="0.254" layer="1"/>
+<wire x1="65.50025" y1="10.69975" x2="65.50025" y2="13.9065" width="0.254" layer="1"/>
 <wire x1="72.194" y1="5.646" x2="72.194" y2="5.929" width="0.127" layer="1"/>
-<wire x1="49.784" y1="14.06525" x2="49.784" y2="11.684" width="0.254" layer="1"/>
-<wire x1="49.784" y1="11.684" x2="50.038" y2="11.43" width="0.254" layer="1"/>
-<wire x1="50.038" y1="11.43" x2="62.738" y2="11.43" width="0.254" layer="1"/>
-<wire x1="62.738" y1="11.43" x2="62.992" y2="11.176" width="0.254" layer="1"/>
-<wire x1="62.992" y1="11.176" x2="63.754" y2="11.176" width="0.254" layer="1"/>
+<wire x1="24.0665" y1="16.60525" x2="43.33875" y2="16.60525" width="0.254" layer="16"/>
+<wire x1="43.33875" y1="16.60525" x2="47.244" y2="12.7" width="0.254" layer="16"/>
+<wire x1="47.244" y1="12.7" x2="49.53" y2="12.7" width="0.254" layer="16"/>
+<wire x1="50.038" y1="13.208" x2="65.024" y2="13.208" width="0.254" layer="16"/>
+<wire x1="65.024" y1="13.208" x2="65.50025" y2="13.68425" width="0.254" layer="16"/>
+<wire x1="65.50025" y1="13.68425" x2="65.50025" y2="13.9065" width="0.254" layer="16"/>
+<wire x1="49.53" y1="12.7" x2="50.038" y2="13.208" width="0.254" layer="16"/>
 </signal>
 <signal name="BATT">
